Commit message: feat:vision 정렬 및 칩 2단 적층 구현

File: src/robot_system_description/urdf/materials.xacro (robot description, xacro)
@@ -4,3 +4,6 @@
   <color rgba="0.700 0.700 0.700 1.000"/>
 </material>
+<material name="black">
+  <color rgba="0.020 0.020 0.020 1.000"/>
+</material>
 </robot>

File: src/robot_system_description/urdf/robot_system.xacro (robot description, xacro)
@@ -18,5 +18,5 @@
       <mesh filename="package://robot_system_description/meshes/base_link.stl" scale="0.001 0.001 0.001"/>
     </geometry>
-    <material name="silver"/>
+    <material name="black"/>
   </visual>
   <collision>
@@ -36,6 +36,6 @@
   <inertial>
     <origin xyz="0.030000000000000013 0.0 0.0" rpy="0 0 0"/>
-    <mass value="7.0649999999999995"/>
-    <inertia ixx="0.038916" iyy="0.038916" izz="0.004239" ixy="-0.0" iyz="0.0" ixz="0.0"/>
+    <mass value="0.18"/>
+    <inertia ixx="0.000991490446" iyy="0.000991490446" izz="0.000108" ixy="0.0" iyz="0.0" ixz="0.0"/>
   </inertial>
   <visual>
@@ -56,6 +56,6 @@
   <inertial>
     <origin xyz="0.030000000000000013 -3.947459643111668e-18 0.0" rpy="0 0 0"/>
-    <mass value="0.5651999999999999"/>
-    <inertia ixx="0.000188" iyy="0.000188" izz="0.000339" ixy="0.0" iyz="0.0" ixz="0.0"/>
+    <mass value="0.09"/>
+    <inertia ixx="0.000029936306" iyy="0.000029936306" izz="0.000053980892" ixy="0.0" iyz="0.0" ixz="0.0"/>
   </inertial>
   <visual>
@@ -76,6 +76,6 @@
   <inertial>
     <origin xyz="0.0001732869481511634 -1.9700445167097035e-18 -0.0303093012095626" rpy="0 0 0"/>
-    <mass value="0.07078216289539181"/>
-    <inertia ixx="1.2e-05" iyy="1e-05" izz="6e-06" ixy="-0.0" iyz="0.0" ixz="0.0"/>
+    <mass value="0.05"/>
+    <inertia ixx="0.000008476712" iyy="0.000007063927" izz="0.000004238356" ixy="0.0" iyz="0.0" ixz="0.0"/>
   </inertial>
   <visual>
@@ -86,14 +86,8 @@
     <material name="silver"/>
   </visual>
-  <collision>
-    <origin xyz="-0.14 0.0 -0.215" rpy="0 0 0"/>
-    <geometry>
-      <mesh filename="package://robot_system_description/meshes/theta_link_1.stl" scale="0.001 0.001 0.001"/>
-    </geometry>
-  </collision>
   <collision name="picker_contact_collision">
-    <origin xyz="0 0 -0.0595" rpy="0 0 0"/>
-    <geometry>
-      <box size="0.012 0.012 0.001"/>
+    <origin xyz="0 0 -0.045" rpy="0 0 0"/>
+    <geometry>
+      <cylinder radius="0.0035" length="0.010"/>
     </geometry>
   </collision>
@@ -102,6 +96,6 @@
   <inertial>
     <origin xyz="8.91814442532711e-18 0.55 0.07933333333333334" rpy="0 0 0"/>
-    <mass value="35.324999999999996"/>
-    <inertia ixx="3.728361" iyy="0.035388" izz="3.751849" ixy="0.0" iyz="0.0" ixz="0.0"/>
+    <mass value="0.45"/>
+    <inertia ixx="0.04749504459" iyy="0.000450802548" izz="0.04779425478" ixy="0.0" iyz="0.0" ixz="0.0"/>
   </inertial>
   <visual>
@@ -124,6 +118,6 @@
   <child link="y_link_1"/>
   <axis xyz="0.0 -1.0 0.0"/>
-  <limit upper="0.4" lower="-0.4" effort="30" velocity="0.2"/>
-  <dynamics damping="25.0" friction="2.0"/>
+  <limit upper="0.4" lower="-0.4" effort="8" velocity="0.2"/>
+  <dynamics damping="3.0" friction="0.0"/>
 </joint>
 <joint name="joint_z" type="prismatic">
@@ -132,6 +126,6 @@
   <child link="z_link_1"/>
   <axis xyz="0.0 0.0 1.0"/>
-  <limit upper="0.115" lower="-0.115" effort="80" velocity="0.25"/>
-  <dynamics damping="3.0" friction="0.05"/>
+  <limit upper="0.115" lower="-0.115" effort="6" velocity="0.25"/>
+  <dynamics damping="0.8" friction="0.0"/>
 </joint>
 <joint name="joint_theta" type="continuous">
@@ -140,5 +134,6 @@
   <child link="theta_link_1"/>
   <axis xyz="-0.0 0.0 -1.0"/>
-  <dynamics damping="0.2" friction="0.05"/>
+  <limit effort="0.2" velocity="3.14"/>
+  <dynamics damping="0.0002" friction="0.0"/>
 </joint>
 <joint name="joint_x" type="prismatic">
@@ -147,12 +142,17 @@
   <child link="x_link_1"/>
   <axis xyz="1.0 0.0 0.0"/>
-  <limit upper="0.4" lower="-0.4" effort="40" velocity="0.2"/>
-  <dynamics damping="30.0" friction="2.0"/>
-</joint>
-<gazebo reference="theta_link_1">
+  <limit upper="0.4" lower="-0.4" effort="12" velocity="0.2"/>
+  <dynamics damping="6.0" friction="0.0"/>
+</joint>
+<gazebo reference="theta_link_1">
+  <selfCollide>true</selfCollide>
+  <kp>1000000.0</kp>
+  <kd>100.0</kd>
+  <maxVel>0.01</maxVel>
+  <minDepth>0.0</minDepth>
   <sensor name="picker_contact_sensor" type="contact">
     <topic>/model/robot_system/picker/contact</topic>
     <contact>
-      <collision>theta_link_1_fixed_joint_lump__picker_contact_collision_collision_1</collision>
+      <collision>theta_link_1_fixed_joint_lump__picker_contact_collision_collision</collision>
     </contact>
     <always_on>1</always_on>
@@ -162,5 +162,5 @@
 <gazebo reference="theta_link_1">
   <sensor type="camera" name="macro_camera">
-    <update_rate>30.0</update_rate>
+    <update_rate>5.0</update_rate>
     <topic>vision/macro_camera/image_raw</topic>
     <camera>
@@ -182,5 +182,5 @@
 <gazebo reference="theta_link_1">
   <sensor type="camera" name="micro_camera_1">
-    <update_rate>30.0</update_rate>
+    <update_rate>5.0</update_rate>
     <topic>vision/micro_camera_1/image_raw</topic>
     <camera>
@@ -202,5 +202,5 @@
 <gazebo reference="theta_link_1">
   <sensor type="camera" name="micro_camera_2">
-    <update_rate>30.0</update_rate>
+    <update_rate>5.0</update_rate>
     <topic>vision/micro_camera_2/image_raw</topic>
     <camera>
@@ -222,5 +222,5 @@
 <gazebo reference="theta_link_1">
   <sensor type="camera" name="micro_camera_3">
-    <update_rate>30.0</update_rate>
+    <update_rate>5.0</update_rate>
     <topic>vision/micro_camera_3/image_raw</topic>
     <camera>
@@ -242,5 +242,5 @@
 <gazebo reference="theta_link_1">
   <sensor type="camera" name="micro_camera_4">
-    <update_rate>30.0</update_rate>
+    <update_rate>5.0</update_rate>
     <topic>vision/micro_camera_4/image_raw</topic>
     <camera>
@@ -273,7 +273,9 @@
     <joint_name>joint_x</joint_name>
     <topic>/model/robot_system/joint/joint_x/cmd_pos</topic>
-    <p_gain>650.0</p_gain>
-    <i_gain>8.0</i_gain>
-    <d_gain>75.0</d_gain>
+    <p_gain>220.0</p_gain>
+    <i_gain>0.0</i_gain>
+    <d_gain>20.0</d_gain>
+    <cmd_max>12.0</cmd_max>
+    <cmd_min>-12.0</cmd_min>
   </plugin>
   <plugin filename="libignition-gazebo-joint-position-controller-system.so"
@@ -281,7 +283,9 @@
     <joint_name>joint_y</joint_name>
     <topic>/model/robot_system/joint/joint_y/cmd_pos</topic>
-    <p_gain>500.0</p_gain>
-    <i_gain>6.0</i_gain>
-    <d_gain>60.0</d_gain>
+    <p_gain>140.0</p_gain>
+    <i_gain>0.0</i_gain>
+    <d_gain>10.5</d_gain>
+    <cmd_max>8.0</cmd_max>
+    <cmd_min>-8.0</cmd_min>
   </plugin>
   <plugin filename="libignition-gazebo-joint-position-controller-system.so"
@@ -289,25 +293,11 @@
     <joint_name>joint_z</joint_name>
     <topic>/model/robot_system/joint/joint_z/cmd_pos</topic>
-    <p_gain>900.0</p_gain>
-    <i_gain>20.0</i_gain>
-    <d_gain>45.0</d_gain>
-  </plugin>
-  <plugin filename="ignition-gazebo-detachable-joint-system"
-          name="ignition::gazebo::systems::DetachableJoint">
-    <parent_link>theta_link_1</parent_link>
-    <child_model>check_chip</child_model>
-    <child_link>chip_link</child_link>
-    <attach_topic>/model/robot_system/vacuum/attach</attach_topic>
-    <detach_topic>/model/robot_system/vacuum/detach</detach_topic>
-    <output_topic>/model/robot_system/vacuum/state</output_topic>
-  </plugin>
-  <plugin filename="ignition-gazebo-detachable-joint-system"
-          name="ignition::gazebo::systems::DetachableJoint">
-    <parent_link>substrate_link</parent_link>
-    <child_model>check_chip</child_model>
-    <child_link>chip_link</child_link>
-    <attach_topic>/model/robot_system/substrate_bond/attach</attach_topic>
-    <detach_topic>/model/robot_system/substrate_bond/detach</detach_topic>
-    <output_topic>/model/robot_system/substrate_bond/state</output_topic>
+    <p_gain>2600.0</p_gain>
+    <i_gain>1200.0</i_gain>
+    <d_gain>40.0</d_gain>
+    <i_max>3.0</i_max>
+    <i_min>-3.0</i_min>
+    <cmd_max>6.0</cmd_max>
+    <cmd_min>-6.0</cmd_min>
   </plugin>
 </gazebo>
@@ -317,53 +307,10 @@
     <joint_name>joint_theta</joint_name>
     <topic>/model/robot_system/joint/joint_theta/cmd_pos</topic>
-    <p_gain>0.3</p_gain>
+    <p_gain>0.05</p_gain>
     <i_gain>0.0</i_gain>
-    <d_gain>0.03</d_gain>
-  </plugin>
-</gazebo>
-<link name="substrate_link">
-  <visual>
-    <origin xyz="0 0 0" rpy="0 0 0"/>
-    <geometry>
-      <box size="0.02 0.02 0.005"/>
-    </geometry>
-  </visual>
-  <collision>
-    <origin xyz="0 0 0" rpy="0 0 0"/>
-    <geometry>
-      <box size="0.02 0.02 0.005"/>
-    </geometry>
-  </collision>
-  <inertial>
-    <mass value="0.005"/>
-    <origin xyz="0 0 0" rpy="0 0 0"/>
-    <inertia ixx="1e-6" iyy="1e-6" izz="1e-6" ixy="0" ixz="0" iyz="0"/>
-  </inertial>
-</link>
-<joint name="world_to_substrate" type="fixed">
-  <parent link="world"/>
-  <child link="substrate_link"/>
-  <origin xyz="0 0 0.0525" rpy="0 0 0"/>
-</joint>
-<gazebo reference="substrate_link">
-  <sensor name="substrate_contact_sensor" type="contact">
-    <topic>/model/robot_system/substrate/contact</topic>
-    <contact>
-      <collision>substrate_link_collision</collision>
-    </contact>
-    <always_on>1</always_on>
-    <update_rate>100</update_rate>
-  </sensor>
-  <visual>
-    <material>
-      <ambient>1 1 1 1</ambient>
-      <diffuse>1 1 1 1</diffuse>
-      <pbr>
-        <metal>
-          <albedo_map>model://robot_system_description/materials/textures/substrate_pattern.png</albedo_map>
-        </metal>
-      </pbr>
-    </material>
-  </visual>
+    <d_gain>0.0008</d_gain>
+    <cmd_max>0.2</cmd_max>
+    <cmd_min>-0.2</cmd_min>
+  </plugin>
 </gazebo>
 </robot>

File: src/robot_system_description/urdf/robot_system_compiled.urdf (robot description, URDF)
Before this commit: robot robot_system, 7 links, 6 joints
Links:
- removed link substrate_link
- link theta_link_1: mass 0.07078216289539181 -> 0.05; geometry collision cylinder length=0.010 radius=0.0035; visual mesh filename=package://robot_system_description/meshes/theta_link_1.stl scale=0.001 0.001 0.001
- link x_link_1: mass 35.324999999999996 -> 0.45
- link y_link_1: mass 7.0649999999999995 -> 0.18
- link z_link_1: mass 0.5651999999999999 -> 0.09
Joints:
- removed joint world_to_substrate
- joint joint_theta: limit (none) -> effort=0.2 velocity=3.14
- joint joint_x: limit lower=-0.4 upper=0.4 effort=40 velocity=0.2 -> lower=-0.4 upper=0.4 effort=12 velocity=0.2
- joint joint_y: limit lower=-0.4 upper=0.4 effort=30 velocity=0.2 -> lower=-0.4 upper=0.4 effort=8 velocity=0.2
- joint joint_z: limit lower=-0.115 upper=0.115 effort=80 velocity=0.25 -> lower=-0.115 upper=0.115 effort=6 velocity=0.25
