Commit message: fix: 로봇 모션 제어 수정

File: src/robot_system_description/urdf/robot_system.xacro (robot description, xacro)
@@ -112,5 +112,6 @@
   <child link="y_link_1"/>
   <axis xyz="0.0 -1.0 0.0"/>
-  <limit upper="0.4" lower="-0.4" effort="100" velocity="100"/>
+  <limit upper="0.4" lower="-0.4" effort="30" velocity="0.2"/>
+  <dynamics damping="25.0" friction="2.0"/>
 </joint>
 <joint name="joint_z" type="prismatic">
@@ -119,5 +120,6 @@
   <child link="z_link_1"/>
   <axis xyz="0.0 0.0 1.0"/>
-  <limit upper="0.1" lower="-0.115" effort="100" velocity="100"/>
+  <limit upper="0.1" lower="-0.115" effort="80" velocity="0.25"/>
+  <dynamics damping="3.0" friction="0.05"/>
 </joint>
 <joint name="joint_theta" type="continuous">
@@ -126,4 +128,5 @@
   <child link="theta_link_1"/>
   <axis xyz="-0.0 0.0 -1.0"/>
+  <dynamics damping="0.2" friction="0.05"/>
 </joint>
 <joint name="joint_x" type="prismatic">
@@ -132,5 +135,6 @@
   <child link="x_link_1"/>
   <axis xyz="1.0 0.0 0.0"/>
-  <limit upper="0.4" lower="-0.4" effort="100" velocity="100"/>
+  <limit upper="0.4" lower="-0.4" effort="40" velocity="0.2"/>
+  <dynamics damping="30.0" friction="2.0"/>
 </joint>
 <gazebo reference="theta_link_1">
@@ -239,7 +243,7 @@
     <joint_name>joint_x</joint_name>
     <topic>/model/robot_system/joint/joint_x/cmd_pos</topic>
-    <p_gain>1000.0</p_gain>
+    <p_gain>30.0</p_gain>
     <i_gain>0.0</i_gain>
-    <d_gain>50.0</d_gain>
+    <d_gain>8.0</d_gain>
   </plugin>
   <plugin filename="libignition-gazebo-joint-position-controller-system.so"
@@ -247,7 +251,7 @@
     <joint_name>joint_y</joint_name>
     <topic>/model/robot_system/joint/joint_y/cmd_pos</topic>
-    <p_gain>300.0</p_gain>
+    <p_gain>25.0</p_gain>
     <i_gain>0.0</i_gain>
-    <d_gain>15.0</d_gain>
+    <d_gain>7.0</d_gain>
   </plugin>
   <plugin filename="libignition-gazebo-joint-position-controller-system.so"
@@ -255,7 +259,7 @@
     <joint_name>joint_z</joint_name>
     <topic>/model/robot_system/joint/joint_z/cmd_pos</topic>
-    <p_gain>500.0</p_gain>
-    <i_gain>1.0</i_gain>
-    <d_gain>5.0</d_gain>
+    <p_gain>80.0</p_gain>
+    <i_gain>0.0</i_gain>
+    <d_gain>8.0</d_gain>
   </plugin>
 </gazebo>
@@ -265,7 +269,7 @@
     <joint_name>joint_theta</joint_name>
     <topic>/model/robot_system/joint/joint_theta/cmd_pos</topic>
-    <p_gain>1.0</p_gain>
+    <p_gain>0.3</p_gain>
     <i_gain>0.0</i_gain>
-    <d_gain>0.1</d_gain>
+    <d_gain>0.03</d_gain>
   </plugin>
 </gazebo>

File: src/robot_system_description/urdf/robot_system_compiled.urdf (robot description, URDF)
Before this commit: robot robot_system, 7 links, 6 joints
Joints:
- joint joint_x: limit lower=-0.4 upper=0.4 effort=100 velocity=100 -> lower=-0.4 upper=0.4 effort=40 velocity=0.2
- joint joint_y: limit lower=-0.4 upper=0.4 effort=100 velocity=100 -> lower=-0.4 upper=0.4 effort=30 velocity=0.2
- joint joint_z: limit lower=-0.115 upper=0.1 effort=100 velocity=100 -> lower=-0.115 upper=0.1 effort=80 velocity=0.25

Commit message: feat: 붉은 칩 추가, micro 카메라 위치 조정통해 광각 보정

File: src/robot_system_description/urdf/robot_system.xacro (robot description, xacro)
@@ -175,5 +175,5 @@
     <always_on>1</always_on>
     <visualize>false</visualize>
-    <pose> 0.0045  0.0045 -0.0505 0 1.5708 1.5708</pose>
+    <pose> 0.006  0.006 -0.0435 0 1.5708 1.5708</pose>
   </sensor>
 </gazebo>
@@ -195,5 +195,5 @@
     <always_on>1</always_on>
     <visualize>false</visualize>
-    <pose> -0.0045  0.0045 -0.0505 0 1.5708 1.5708</pose>
+    <pose> -0.006  0.006 -0.0435 0 1.5708 1.5708</pose>
   </sensor>
 </gazebo>
@@ -215,5 +215,5 @@
     <always_on>1</always_on>
     <visualize>false</visualize>
-    <pose> -0.0045  -0.0045 -0.0505 0 1.5708 1.5708</pose>
+    <pose> -0.006  -0.006 -0.0435 0 1.5708 1.5708</pose>
   </sensor>
 </gazebo>
@@ -235,5 +235,5 @@
     <always_on>1</always_on>
     <visualize>false</visualize>
-    <pose> 0.0045  -0.0045 -0.0505 0 1.5708 1.5708</pose>
+    <pose> 0.006  -0.006 -0.0435 0 1.5708 1.5708</pose>
   </sensor>
 </gazebo>
@@ -332,3 +332,33 @@
   </visual>
 </gazebo>
+<link name="red_check_chip_link">
+  <visual>
+    <origin xyz="0 0 0" rpy="0 0 0"/>
+    <geometry>
+      <box size="0.011 0.011 0.0001"/>
+    </geometry>
+    <material name="red_color">
+      <color rgba="1.0 0.0 0.0 1.0"/>
+    </material>
+  </visual>
+  <collision>
+    <origin xyz="0 0 0" rpy="0 0 0"/>
+    <geometry>
+      <box size="0.011 0.011 0.0001"/>
+    </geometry>
+  </collision>
+  <inertial>
+    <mass value="0.001"/>
+    <origin xyz="0 0 0" rpy="0 0 0"/>
+    <inertia ixx="1e-8" iyy="1e-8" izz="1e-8" ixy="0" ixz="0" iyz="0"/>
+  </inertial>
+</link>
+<joint name="world_to_red_check_chip" type="fixed">
+  <parent link="world"/>
+  <child link="red_check_chip_link"/>
+  <origin xyz="0.14 0 0.153" rpy="0 0 0"/>
+</joint>
+<gazebo reference="red_check_chip_link">
+  <material>Gazebo/Red</material>
+</gazebo>
 </robot>

File: src/robot_system_description/urdf/robot_system_compiled.urdf (robot description, URDF)
Before this commit: robot robot_system, 7 links, 6 joints
Links:
- added link red_check_chip_link, mass 0.001; collision box size=0.011 0.011 0.0001; visual box size=0.011 0.011 0.0001
Joints:
- added joint world_to_red_check_chip: type fixed, parent world, child red_check_chip_link, origin xyz=0.14 0 0.153 rpy=0 0 0

Commit message: feat:칩 이미지 파일 조정,substrate 추가

File: src/robot_system_description/urdf/robot_system.xacro (robot description, xacro)
@@ -317,5 +317,5 @@
   <parent link="world"/>
   <child link="check_chip_link"/>
-  <origin xyz="0.14 0 0.05005" rpy="0 0 0"/>
+  <origin xyz="0.14 0 0.05505" rpy="0 0 0"/>
 </joint>
 <gazebo reference="check_chip_link">
@@ -362,3 +362,40 @@
   <material>Gazebo/Red</material>
 </gazebo>
+<link name="substrate_link">
+  <visual>
+    <origin xyz="0 0 0" rpy="0 0 0"/>
+    <geometry>
+      <box size="0.02 0.02 0.005"/>
+    </geometry>
+  </visual>
+  <collision>
+    <origin xyz="0 0 0" rpy="0 0 0"/>
+    <geometry>
+      <box size="0.02 0.02 0.005"/>
+    </geometry>
+  </collision>
+  <inertial>
+    <mass value="0.005"/>
+    <origin xyz="0 0 0" rpy="0 0 0"/>
+    <inertia ixx="1e-6" iyy="1e-6" izz="1e-6" ixy="0" ixz="0" iyz="0"/>
+  </inertial>
+</link>
+<joint name="world_to_substrate" type="fixed">
+  <parent link="world"/>
+  <child link="substrate_link"/>
+  <origin xyz="0.14 0 0.0525" rpy="0 0 0"/>
+</joint>
+<gazebo reference="substrate_link">
+  <visual>
+    <material>
+      <ambient>1 1 1 1</ambient>
+      <diffuse>1 1 1 1</diffuse>
+      <pbr>
+        <metal>
+          <albedo_map>model://robot_system_description/materials/textures/substrate_pattern.png</albedo_map>
+        </metal>
+      </pbr>
+    </material>
+  </visual>
+</gazebo>
 </robot>

File: src/robot_system_description/urdf/robot_system_compiled.urdf (robot description, URDF)
Before this commit: robot robot_system, 8 links, 7 joints
Links:
- added link substrate_link, mass 0.005; collision box size=0.02 0.02 0.005; visual box size=0.02 0.02 0.005
Joints:
- added joint world_to_substrate: type fixed, parent world, child substrate_link, origin xyz=0.14 0 0.0525 rpy=0 0 0
- joint world_to_check_chip: origin xyz=0.14 0 0.05005 rpy=0 0 0 -> xyz=0.14 0 0.05505 rpy=0 0 0

Commit message: feat: Gazebo 가동범위 및 그림오류 수정

File: src/robot_system_description/urdf/robot_system.xacro (robot description, xacro)
@@ -120,5 +120,5 @@
   <child link="z_link_1"/>
   <axis xyz="0.0 0.0 1.0"/>
-  <limit upper="0.1" lower="-0.115" effort="80" velocity="0.25"/>
+  <limit upper="0.115" lower="-0.115" effort="80" velocity="0.25"/>
   <dynamics damping="3.0" friction="0.05"/>
 </joint>
@@ -326,5 +326,5 @@
       <pbr>
         <metal>
-         <albedo_map>model://robot_system_description/materials/textures/chip_pattern.jpg</albedo_map>
+         <albedo_map>model://robot_system_description/materials/textures/chip_pattern.png</albedo_map>
         </metal>
       </pbr>

Commit message: feat: stabilize gazebo robot demo control

File: src/robot_system_description/urdf/robot_system.xacro (robot description, xacro)
@@ -239,11 +239,19 @@
 </gazebo>
 <gazebo>
+  <plugin filename="libignition-gazebo-joint-state-publisher-system.so"
+          name="ignition::gazebo::systems::JointStatePublisher">
+    <topic>/model/robot_system/joint_state</topic>
+    <joint_name>joint_x</joint_name>
+    <joint_name>joint_y</joint_name>
+    <joint_name>joint_z</joint_name>
+    <joint_name>joint_theta</joint_name>
+  </plugin>
   <plugin filename="libignition-gazebo-joint-position-controller-system.so"
           name="ignition::gazebo::systems::JointPositionController">
     <joint_name>joint_x</joint_name>
     <topic>/model/robot_system/joint/joint_x/cmd_pos</topic>
-    <p_gain>30.0</p_gain>
-    <i_gain>0.0</i_gain>
-    <d_gain>8.0</d_gain>
+    <p_gain>650.0</p_gain>
+    <i_gain>8.0</i_gain>
+    <d_gain>75.0</d_gain>
   </plugin>
   <plugin filename="libignition-gazebo-joint-position-controller-system.so"
@@ -251,7 +259,7 @@
     <joint_name>joint_y</joint_name>
     <topic>/model/robot_system/joint/joint_y/cmd_pos</topic>
-    <p_gain>25.0</p_gain>
-    <i_gain>0.0</i_gain>
-    <d_gain>7.0</d_gain>
+    <p_gain>500.0</p_gain>
+    <i_gain>6.0</i_gain>
+    <d_gain>60.0</d_gain>
   </plugin>
   <plugin filename="libignition-gazebo-joint-position-controller-system.so"
@@ -259,7 +267,7 @@
     <joint_name>joint_z</joint_name>
     <topic>/model/robot_system/joint/joint_z/cmd_pos</topic>
-    <p_gain>80.0</p_gain>
-    <i_gain>0.0</i_gain>
-    <d_gain>8.0</d_gain>
+    <p_gain>900.0</p_gain>
+    <i_gain>20.0</i_gain>
+    <d_gain>45.0</d_gain>
   </plugin>
 </gazebo>
@@ -326,39 +334,9 @@
       <pbr>
         <metal>
-         <albedo_map>model://robot_system_description/materials/textures/chip_pattern.png</albedo_map>
+          <albedo_map>model://robot_system_description/materials/textures/chip_pattern.png</albedo_map>
         </metal>
       </pbr>
     </material>
   </visual>
-</gazebo>
-<link name="red_check_chip_link">
-  <visual>
-    <origin xyz="0 0 0" rpy="0 0 0"/>
-    <geometry>
-      <box size="0.011 0.011 0.0001"/>
-    </geometry>
-    <material name="red_color">
-      <color rgba="1.0 0.0 0.0 1.0"/>
-    </material>
-  </visual>
-  <collision>
-    <origin xyz="0 0 0" rpy="0 0 0"/>
-    <geometry>
-      <box size="0.011 0.011 0.0001"/>
-    </geometry>
-  </collision>
-  <inertial>
-    <mass value="0.001"/>
-    <origin xyz="0 0 0" rpy="0 0 0"/>
-    <inertia ixx="1e-8" iyy="1e-8" izz="1e-8" ixy="0" ixz="0" iyz="0"/>
-  </inertial>
-</link>
-<joint name="world_to_red_check_chip" type="fixed">
-  <parent link="world"/>
-  <child link="red_check_chip_link"/>
-  <origin xyz="0.14 0 0.153" rpy="0 0 0"/>
-</joint>
-<gazebo reference="red_check_chip_link">
-  <material>Gazebo/Red</material>
 </gazebo>
 <link name="substrate_link">

File: src/robot_system_description/urdf/robot_system_compiled.urdf (robot description, URDF)
Before this commit: robot robot_system, 9 links, 8 joints
Links:
- removed link red_check_chip_link
Joints:
- removed joint world_to_red_check_chip

Commit message: feat:그리퍼 동작 메커니즘 개선

File: src/robot_system_description/urdf/robot_system.xacro (robot description, xacro)
@@ -86,4 +86,10 @@
     </geometry>
   </collision>
+  <collision name="picker_contact_collision">
+    <origin xyz="0 0 -0.1645" rpy="0 0 0"/>
+    <geometry>
+      <box size="0.012 0.012 0.001"/>
+    </geometry>
+  </collision>
 </link>
 <link name="x_link_1">
@@ -138,4 +144,14 @@
   <dynamics damping="30.0" friction="2.0"/>
 </joint>
+<gazebo reference="theta_link_1">
+  <sensor name="picker_contact_sensor" type="contact">
+    <contact>
+      <collision>picker_contact_collision</collision>
+      <topic>/model/robot_system/picker/contact</topic>
+    </contact>
+    <always_on>1</always_on>
+    <update_rate>100</update_rate>
+  </sensor>
+</gazebo>
 <gazebo reference="theta_link_1">
   <sensor type="camera" name="macro_camera">
@@ -271,4 +287,13 @@
     <d_gain>45.0</d_gain>
   </plugin>
+  <plugin filename="ignition-gazebo-detachable-joint-system"
+          name="ignition::gazebo::systems::DetachableJoint">
+    <parent_link>theta_link_1</parent_link>
+    <child_model>check_chip</child_model>
+    <child_link>chip_link</child_link>
+    <attach_topic>/model/robot_system/vacuum/attach</attach_topic>
+    <detach_topic>/model/robot_system/vacuum/detach</detach_topic>
+    <output_topic>/model/robot_system/vacuum/state</output_topic>
+  </plugin>
 </gazebo>
 <gazebo>
@@ -282,56 +307,4 @@
   </plugin>
 </gazebo>
-<gazebo reference="theta_link_1">
-  <light name="gripper_led" type="point">
-    <pose>0 0 -0.05 0 0 0</pose>
-    <diffuse>1.0 1.0 1.0 1.0</diffuse>
-    <specular>1.0 1.0 1.0 1.0</specular>
-    <visualize>false</visualize>
-    <attenuation>
-      <range>2.0</range>
-      <constant>1.0</constant>
-      <linear>0.005</linear>
-      <quadratic>0.001</quadratic>
-    </attenuation>
-    <cast_shadows>false</cast_shadows>
-  </light>
-</gazebo>
-<link name="check_chip_link">
-  <visual>
-    <origin xyz="0 0 0" rpy="0 0 0"/>
-    <geometry>
-      <box size="0.011 0.011 0.0001"/>
-    </geometry>
-  </visual>
-  <collision>
-    <origin xyz="0 0 0" rpy="0 0 0"/>
-    <geometry>
-      <box size="0.011 0.011 0.0001"/>
-    </geometry>
-  </collision>
-  <inertial>
-    <mass value="0.001"/>
-    <origin xyz="0 0 0" rpy="0 0 0"/>
-    <inertia ixx="1e-8" iyy="1e-8" izz="1e-8" ixy="0" ixz="0" iyz="0"/>
-  </inertial>
-</link>
-<joint name="world_to_check_chip" type="fixed">
-  <parent link="world"/>
-  <child link="check_chip_link"/>
-  <origin xyz="0.14 0 0.05505" rpy="0 0 0"/>
-</joint>
-<gazebo reference="check_chip_link">
-  <visual>
-    <material>
-      <ambient>1 1 1 1</ambient>
-      <diffuse>1 1 1 1</diffuse>
-      <pbr>
-        <metal>
-          <albedo_map>model://robot_system_description/materials/textures/chip_pattern.png</albedo_map>
-        </metal>
-      </pbr>
-    </material>
-  </visual>
-</gazebo>
 <link name="substrate_link">
   <visual>
@@ -356,5 +329,5 @@
   <parent link="world"/>
   <child link="substrate_link"/>
-  <origin xyz="0.14 0 0.0525" rpy="0 0 0"/>
+  <origin xyz="0 0 0.0525" rpy="0 0 0"/>
 </joint>
 <gazebo reference="substrate_link">

File: src/robot_system_description/urdf/robot_system_compiled.urdf (robot description, URDF)
Before this commit: robot robot_system, 8 links, 7 joints
Links:
- removed link check_chip_link
- link theta_link_1: geometry collision box size=0.012 0.012 0.001; collision mesh filename=package://robot_system_description/meshes/theta_link_1.stl scale=0.001 0.001 0.001
Joints:
- removed joint world_to_check_chip
- joint joint_z: limit lower=-0.115 upper=0.1 effort=80 velocity=0.25 -> lower=-0.115 upper=0.115 effort=80 velocity=0.25
- joint world_to_substrate: origin xyz=0.14 0 0.0525 rpy=0 0 0 -> xyz=0 0 0.0525 rpy=0 0 0

Commit message: feat:그래퍼 좌표 및 매커니즘 개선

File: src/robot_system_description/urdf/robot_system.xacro (robot description, xacro)
@@ -26,4 +26,10 @@
     </geometry>
   </collision>
+  <collision name="base_work_surface_collision">
+    <origin xyz="0 0 0.0495" rpy="0 0 0"/>
+    <geometry>
+      <box size="1.2 1.2 0.001"/>
+    </geometry>
+  </collision>
 </link>
 <link name="y_link_1">
@@ -87,5 +93,5 @@
   </collision>
   <collision name="picker_contact_collision">
-    <origin xyz="0 0 -0.1645" rpy="0 0 0"/>
+    <origin xyz="0 0 -0.0595" rpy="0 0 0"/>
     <geometry>
       <box size="0.012 0.012 0.001"/>
@@ -146,7 +152,7 @@
 <gazebo reference="theta_link_1">
   <sensor name="picker_contact_sensor" type="contact">
+    <topic>/model/robot_system/picker/contact</topic>
     <contact>
-      <collision>picker_contact_collision</collision>
-      <topic>/model/robot_system/picker/contact</topic>
+      <collision>theta_link_1_fixed_joint_lump__picker_contact_collision_collision_1</collision>
     </contact>
     <always_on>1</always_on>
@@ -296,4 +302,13 @@
     <output_topic>/model/robot_system/vacuum/state</output_topic>
   </plugin>
+  <plugin filename="ignition-gazebo-detachable-joint-system"
+          name="ignition::gazebo::systems::DetachableJoint">
+    <parent_link>substrate_link</parent_link>
+    <child_model>check_chip</child_model>
+    <child_link>chip_link</child_link>
+    <attach_topic>/model/robot_system/substrate_bond/attach</attach_topic>
+    <detach_topic>/model/robot_system/substrate_bond/detach</detach_topic>
+    <output_topic>/model/robot_system/substrate_bond/state</output_topic>
+  </plugin>
 </gazebo>
 <gazebo>
@@ -332,4 +347,12 @@
 </joint>
 <gazebo reference="substrate_link">
+  <sensor name="substrate_contact_sensor" type="contact">
+    <topic>/model/robot_system/substrate/contact</topic>
+    <contact>
+      <collision>substrate_link_collision</collision>
+    </contact>
+    <always_on>1</always_on>
+    <update_rate>100</update_rate>
+  </sensor>
   <visual>
     <material>

File: src/robot_system_description/urdf/robot_system_compiled.urdf (robot description, URDF)
Before this commit: robot robot_system, 7 links, 6 joints
Links:
- link base_link: geometry collision box size=1.2 1.2 0.001; collision mesh filename=package://robot_system_description/meshes/base_link.stl scale=0.001 0.001 0.001

Commit message: feat:정렬 chip 4 ~ 16개 파라미터 의존 개선

File: src/robot_system_description/urdf/robot_system.xacro (robot description, xacro)
@@ -118,5 +118,5 @@
   <child link="y_link_1"/>
   <axis xyz="0.0 -1.0 0.0"/>
-  <limit upper="0.4" lower="-0.4" effort="8" velocity="0.2"/>
+  <limit upper="0.405" lower="-0.405" effort="8" velocity="0.2"/>
   <dynamics damping="3.0" friction="0.0"/>
 </joint>
@@ -157,10 +157,10 @@
     </contact>
     <always_on>1</always_on>
-    <update_rate>100</update_rate>
+    <update_rate>50</update_rate>
   </sensor>
 </gazebo>
 <gazebo reference="theta_link_1">
   <sensor type="camera" name="macro_camera">
-    <update_rate>5.0</update_rate>
+    <update_rate>2.0</update_rate>
     <topic>vision/macro_camera/image_raw</topic>
     <camera>
@@ -175,5 +175,5 @@
       </clip>
     </camera>
-    <always_on>1</always_on>
+    <always_on>0</always_on>
     <visualize>false</visualize>
     <pose>0.0125 0 -0.038 0 1.5708 1.5708</pose>
@@ -182,5 +182,5 @@
 <gazebo reference="theta_link_1">
   <sensor type="camera" name="micro_camera_1">
-    <update_rate>5.0</update_rate>
+    <update_rate>2.0</update_rate>
     <topic>vision/micro_camera_1/image_raw</topic>
     <camera>
@@ -195,5 +195,5 @@
       </clip>
     </camera>
-    <always_on>1</always_on>
+    <always_on>0</always_on>
     <visualize>false</visualize>
     <pose> 0.006  0.006 -0.0435 0 1.5708 1.5708</pose>
@@ -202,5 +202,5 @@
 <gazebo reference="theta_link_1">
   <sensor type="camera" name="micro_camera_2">
-    <update_rate>5.0</update_rate>
+    <update_rate>2.0</update_rate>
     <topic>vision/micro_camera_2/image_raw</topic>
     <camera>
@@ -215,5 +215,5 @@
       </clip>
     </camera>
-    <always_on>1</always_on>
+    <always_on>0</always_on>
     <visualize>false</visualize>
     <pose> -0.006  0.006 -0.0435 0 1.5708 1.5708</pose>
@@ -222,5 +222,5 @@
 <gazebo reference="theta_link_1">
   <sensor type="camera" name="micro_camera_3">
-    <update_rate>5.0</update_rate>
+    <update_rate>2.0</update_rate>
     <topic>vision/micro_camera_3/image_raw</topic>
     <camera>
@@ -235,5 +235,5 @@
       </clip>
     </camera>
-    <always_on>1</always_on>
+    <always_on>0</always_on>
     <visualize>false</visualize>
     <pose> -0.006  -0.006 -0.0435 0 1.5708 1.5708</pose>
@@ -242,5 +242,5 @@
 <gazebo reference="theta_link_1">
   <sensor type="camera" name="micro_camera_4">
-    <update_rate>5.0</update_rate>
+    <update_rate>2.0</update_rate>
     <topic>vision/micro_camera_4/image_raw</topic>
     <camera>
@@ -255,5 +255,5 @@
       </clip>
     </camera>
-    <always_on>1</always_on>
+    <always_on>0</always_on>
     <visualize>false</visualize>
     <pose> 0.006  -0.006 -0.0435 0 1.5708 1.5708</pose>

File: src/robot_system_description/urdf/robot_system_compiled.urdf (robot description, URDF)
Before this commit: robot robot_system, 6 links, 5 joints
Joints:
- joint joint_y: limit lower=-0.4 upper=0.4 effort=8 velocity=0.2 -> lower=-0.405 upper=0.405 effort=8 velocity=0.2
